Commit message: Feature: Octomap and Gripper fix

File: kortex_description/grippers/robotiq_2f_85/urdf/robotiq_2f_85_transmission_macro.xacro (robot description, xacro)
@@ -19,4 +19,5 @@
                 <offset>0.0</offset>
                 <maxEffort>5.0</maxEffort>
+		<hasPID />
             </plugin>
             <plugin filename="libroboticsgroup_gazebo_mimic_joint_plugin.so" name="mimic_robotiq_85_2">
@@ -26,4 +27,5 @@
                 <offset>0.0</offset>
                 <maxEffort>5.0</maxEffort>
+		<hasPID />
             </plugin>
             <plugin filename="libroboticsgroup_gazebo_mimic_joint_plugin.so" name="mimic_robotiq_85_3">
@@ -33,4 +35,5 @@
                 <offset>0.0</offset>
                 <maxEffort>5.0</maxEffort>
+		<hasPID />
             </plugin>
             <plugin filename="libroboticsgroup_gazebo_mimic_joint_plugin.so" name="mimic_robotiq_85_4">
@@ -40,4 +43,5 @@
                 <offset>0.0</offset>
                 <maxEffort>5.0</maxEffort>
+		<hasPID />
             </plugin>
             <plugin filename="libroboticsgroup_gazebo_mimic_joint_plugin.so" name="mimic_robotiq_85_5">
@@ -47,4 +51,5 @@
                 <offset>0.0</offset>
                 <maxEffort>5.0</maxEffort>
+		<hasPID />
             </plugin>
             <plugin name="gazebo_grasp_fix" filename="libgazebo_grasp_fix.so">
@@ -55,10 +60,10 @@
                     <gripper_link> right_inner_finger </gripper_link>
                 </arm>
-                <forces_angle_tolerance>100</forces_angle_tolerance>
+                <forces_angle_tolerance>130</forces_angle_tolerance>
                 <update_rate>10</update_rate>
-                <grip_count_threshold>3</grip_count_threshold>
-                <max_grip_count>10</max_grip_count>
+                <grip_count_threshold>1</grip_count_threshold>
+                <max_grip_count>8</max_grip_count>
                 <release_tolerance>0.001</release_tolerance>
-                <disable_collisions_on_attach>false</disable_collisions_on_attach>
+                <disable_collisions_on_attach>true</disable_collisions_on_attach>
                 <contact_topic>__default_topic__</contact_topic>
             </plugin>

File: kortex_description/grippers/robotiq_2f_85/urdf/robotiq_arg2f_85_model_macro.xacro (robot description, xacro)
@@ -143,9 +143,9 @@
   <xacro:macro name="inner_finger_joint" params="prefix fingerprefix">
     <joint name="${prefix}${fingerprefix}_inner_finger_joint" type="revolute">
-      <origin xyz="0 0.0061 0.0471" rpy="0 0 0"/>
+      <origin xyz="0 0 0.05" rpy="0 0 0"/>
       <parent link="${prefix}${fingerprefix}_outer_finger" />
       <child link="${prefix}${fingerprefix}_inner_finger" />
       <axis xyz="1 0 0" />
-      <limit lower="-0.8757" upper="0.8757" velocity="2.0" effort="1000" />
+      <limit lower="-0.81" upper="0.81" velocity="2.0" effort="1000" />
       <mimic joint="${prefix}finger_joint" multiplier="-1" offset="0" />
     </joint>
@@ -153,5 +153,5 @@
   <xacro:macro name="inner_finger_pad_joint" params="prefix fingerprefix">
     <joint name="${prefix}${fingerprefix}_inner_finger_pad_joint" type="fixed">
-      <origin xyz="0 -0.0220203446692936 0.03242" rpy="0 0 0"/>
+      <origin xyz="0 -0.022 0.032" rpy="0 0 0"/>
       <parent link="${prefix}${fingerprefix}_inner_finger" />
       <child link="${prefix}${fingerprefix}_inner_finger_pad" />
